Commit message: basic transform of gap point from left_camera_link to floor_frame

File: urdf/wombot.urdf.xacro (robot description, xacro)
@@ -77,4 +77,10 @@
     <child link="base_footprint" />
   </joint>
+  <link name="floor"/>
+  <joint name="floor_joint" type="fixed">
+    <origin xyz="0 0 -0.02085" rpy="0 0 0" />
+    <parent link="left_camera_link" />
+    <child link="floor" />
+  </joint>
   <!-- Inertial link stores the robot's inertial information -->
   <link name="inertial_link">

Commit message: fixed transform for floor frame to left_camera_link (not finished though)

File: urdf/wombot.urdf.xacro (robot description, xacro)
@@ -22,11 +22,11 @@
   <!-- Wheel Mounting Positions -->
   <!-- TODO: Insert real values -->
-  <xacro:property name="wheelbase"		value="0.200" />
-  <xacro:property name="track"			value="0.240" />
-  <xacro:property name="caster_track"			value="0.220" />
+  <xacro:property name="wheelbase"		value="0.2159" />
+  <xacro:property name="track"			value="0.196825" />
+  <xacro:property name="caster_track"			value="0.196825" />
   <xacro:property name="ground_clearance"	value="0.00635" />
   <xacro:property name="front_axle_x_offset"	value="0.09" />
-  <xacro:property name="caster_wheel_vertical_offset"	value="0.015" />
-  <xacro:property name="rear_axle_x_offset"	value="-0.09" />
+    <xacro:property name="rear_axle_x_offset"	value="-0.09" />
+  <!-- <xacro:property name="caster_wheel_vertical_offset"	value="0.015" /> -->
   <!-- Wheel Properties -->
   <xacro:property name="drive_wheel_length" value="0.03" />
@@ -79,5 +79,7 @@
   <link name="floor"/>
   <joint name="floor_joint" type="fixed">
+  <!-- intrinsic meaning it rotates about whatever the nex axes direction is -->
     <origin xyz="0 0 -0.02085" rpy="0 0 0" />
+    <!-- <origin xyz="0 0 -0.02085" rpy="1.57 0 1.57" /> -->
     <parent link="left_camera_link" />
     <child link="floor" />
